File: Hardware/io2.kicad_sch (KiCad schematic)
At the start: 15 parts, among them U1 H616, Y1 25MHz

Commit message: added testpoint for TX/RX and updated readme
Parts:
- Y1: value 25MHz -> 24MHz
Changed lines of the file:
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@@
     (pin "1")
     (instances
-      (project "H616_devboard"
+      (project "kryptokrona-mini-miner"
         (path "/44f68964-8d75-4db0-b784-705712e148bc/5d9fa4e3-c1a9-47c1-b361-a7aa11440b42"
           (reference "#PWR076") (unit 1)
@@
     (pin "1")
     (instances
-      (project "H616_devboard"
+      (project "kryptokrona-mini-miner"
         (path "/44f68964-8d75-4db0-b784-705712e148bc/5d9fa4e3-c1a9-47c1-b361-a7aa11440b42"
           (reference "#PWR085") (unit 1)
@@
     (pin "2")
     (instances
-      (project "H616_devboard"
+      (project "kryptokrona-mini-miner"
         (path "/44f68964-8d75-4db0-b784-705712e148bc/5d9fa4e3-c1a9-47c1-b361-a7aa11440b42"
           (reference "C59") (unit 1)
@@
     (pin "2")
     (instances
-      (project "H616_devboard"
+      (project "kryptokrona-mini-miner"
         (path "/44f68964-8d75-4db0-b784-705712e148bc/5d9fa4e3-c1a9-47c1-b361-a7aa11440b42"
           (reference "R19") (unit 1)
@@
     (pin "1")
     (instances
-      (project "H616_devboard"
+      (project "kryptokrona-mini-miner"
         (path "/44f68964-8d75-4db0-b784-705712e148bc/5d9fa4e3-c1a9-47c1-b361-a7aa11440b42"
           (reference "#PWR071") (unit 1)
@@
     (pin "1")
     (instances
-      (project "H616_devboard"
+      (project "kryptokrona-mini-miner"
         (path "/44f68964-8d75-4db0-b784-705712e148bc/5d9fa4e3-c1a9-47c1-b361-a7aa11440b42"
           (reference "#PWR069") (unit 1)
@@
     (pin "2")
     (instances
-      (project "H616_devboard"
+      (project "kryptokrona-mini-miner"
         (path "/44f68964-8d75-4db0-b784-705712e148bc/5d9fa4e3-c1a9-47c1-b361-a7aa11440b42"
           (reference "C64") (unit 1)
@@
     (pin "1")
     (instances
-      (project "H616_devboard"
+      (project "kryptokrona-mini-miner"
         (path "/44f68964-8d75-4db0-b784-705712e148bc/5d9fa4e3-c1a9-47c1-b361-a7aa11440b42"
           (reference "#PWR081") (unit 1)
@@
     (pin "2")
     (instances
-      (project "H616_devboard"
+      (project "kryptokrona-mini-miner"
         (path "/44f68964-8d75-4db0-b784-705712e148bc/5d9fa4e3-c1a9-47c1-b361-a7aa11440b42"
           (reference "C58") (unit 1)
@@
     (pin "1")
     (instances
-      (project "H616_devboard"
+      (project "kryptokrona-mini-miner"
         (path "/44f68964-8d75-4db0-b784-705712e148bc/5d9fa4e3-c1a9-47c1-b361-a7aa11440b42"
           (reference "#PWR078") (unit 1)
@@
     (pin "1")
     (instances
-      (project "H616_devboard"
+      (project "kryptokrona-mini-miner"
         (path "/44f68964-8d75-4db0-b784-705712e148bc/5d9fa4e3-c1a9-47c1-b361-a7aa11440b42"
           (reference "#PWR079") (unit 1)
@@
     (pin "1")
     (instances
-      (project "H616_devboard"
+      (project "kryptokrona-mini-miner"
         (path "/44f68964-8d75-4db0-b784-705712e148bc/5d9fa4e3-c1a9-47c1-b361-a7aa11440b42"
           (reference "#PWR072") (unit 1)
@@
     (pin "2")
     (instances
-      (project "H616_devboard"
+      (project "kryptokrona-mini-miner"
         (path "/44f68964-8d75-4db0-b784-705712e148bc/5d9fa4e3-c1a9-47c1-b361-a7aa11440b42"
           (reference "C63") (unit 1)
@@
     (pin "1")
     (instances
-      (project "H616_devboard"
+      (project "kryptokrona-mini-miner"
         (path "/44f68964-8d75-4db0-b784-705712e148bc/5d9fa4e3-c1a9-47c1-b361-a7aa11440b42"
           (reference "#PWR075") (unit 1)
@@
     (pin "1")
     (instances
-      (project "H616_devboard"
+      (project "kryptokrona-mini-miner"
         (path "/44f68964-8d75-4db0-b784-705712e148bc/5d9fa4e3-c1a9-47c1-b361-a7aa11440b42"
           (reference "#PWR070") (unit 1)
@@
       (effects (font (size 1.27 1.27)))
     )
-    (property "Value" "25MHz" (at 140.335 146.685 90)
+    (property "Value" "24MHz" (at 140.335 146.685 90)
       (effects (font (size 1.27 1.27)))
     )
@@
     (pin "4")
     (instances
-      (project "H616_devboard"
+      (project "kryptokrona-mini-miner"
         (path "/44f68964-8d75-4db0-b784-705712e148bc/5d9fa4e3-c1a9-47c1-b361-a7aa11440b42"
           (reference "Y1") (unit 1)
@@
     (pin "2")
     (instances
-      (project "H616_devboard"
+      (project "kryptokrona-mini-miner"
         (path "/44f68964-8d75-4db0-b784-705712e148bc/5d9fa4e3-c1a9-47c1-b361-a7aa11440b42"
           (reference "C57") (unit 1)
@@
     (pin "1")
     (instances
-      (project "H616_devboard"
+      (project "kryptokrona-mini-miner"
         (path "/44f68964-8d75-4db0-b784-705712e148bc/5d9fa4e3-c1a9-47c1-b361-a7aa11440b42"
           (reference "#PWR073") (unit 1)
@@
     (pin "2")
     (instances
-      (project "H616_devboard"
+      (project "kryptokrona-mini-miner"
         (path "/44f68964-8d75-4db0-b784-705712e148bc/5d9fa4e3-c1a9-47c1-b361-a7aa11440b42"
           (reference "C56") (unit 1)
@@
     (pin "1")
     (instances
-      (project "H616_devboard"
+      (project "kryptokrona-mini-miner"
         (path "/44f68964-8d75-4db0-b784-705712e148bc/5d9fa4e3-c1a9-47c1-b361-a7aa11440b42"
           (reference "#PWR074") (unit 1)
@@
     (pin "1")
     (instances
-      (project "H616_devboard"
+      (project "kryptokrona-mini-miner"
         (path "/44f68964-8d75-4db0-b784-705712e148bc/5d9fa4e3-c1a9-47c1-b361-a7aa11440b42"
           (reference "#PWR082") (unit 1)
@@
     (pin "2")
     (instances
-      (project "H616_devboard"
+      (project "kryptokrona-mini-miner"
         (path "/44f68964-8d75-4db0-b784-705712e148bc/5d9fa4e3-c1a9-47c1-b361-a7aa11440b42"
           (reference "C61") (unit 1)
@@
     (pin "1")
     (instances
-      (project "H616_devboard"
+      (project "kryptokrona-mini-miner"
         (path "/44f68964-8d75-4db0-b784-705712e148bc/5d9fa4e3-c1a9-47c1-b361-a7aa11440b42"
           (reference "#PWR077") (unit 1)
@@
     (pin "2")
     (instances
-      (project "H616_devboard"
+      (project "kryptokrona-mini-miner"
         (path "/44f68964-8d75-4db0-b784-705712e148bc/5d9fa4e3-c1a9-47c1-b361-a7aa11440b42"
           (reference "C60") (unit 1)
@@
     (pin "1")
     (instances
-      (project "H616_devboard"
+      (project "kryptokrona-mini-miner"
         (path "/44f68964-8d75-4db0-b784-705712e148bc/5d9fa4e3-c1a9-47c1-b361-a7aa11440b42"
           (reference "#PWR080") (unit 1)
@@
     (pin "2")
     (instances
-      (project "H616_devboard"
+      (project "kryptokrona-mini-miner"
         (path "/44f68964-8d75-4db0-b784-705712e148bc/5d9fa4e3-c1a9-47c1-b361-a7aa11440b42"
           (reference "R20") (unit 1)
@@
     (pin "2")
     (instances
-      (project "H616_devboard"
+      (project "kryptokrona-mini-miner"
         (path "/44f68964-8d75-4db0-b784-705712e148bc/5d9fa4e3-c1a9-47c1-b361-a7aa11440b42"
           (reference "C55") (unit 1)
@@
     (pin "2")
     (instances
-      (project "H616_devboard"
+      (project "kryptokrona-mini-miner"
         (path "/44f68964-8d75-4db0-b784-705712e148bc/5d9fa4e3-c1a9-47c1-b361-a7aa11440b42"
           (reference "C54") (unit 1)
@@
     (pin "1")
     (instances
-      (project "H616_devboard"
+      (project "kryptokrona-mini-miner"
         (path "/44f68964-8d75-4db0-b784-705712e148bc/5d9fa4e3-c1a9-47c1-b361-a7aa11440b42"
           (reference "#PWR068") (unit 1)
@@
     (pin "1")
     (instances
-      (project "H616_devboard"
+      (project "kryptokrona-mini-miner"
         (path "/44f68964-8d75-4db0-b784-705712e148bc/5d9fa4e3-c1a9-47c1-b361-a7aa11440b42"
           (reference "#PWR084") (unit 1)
@@
     (pin "1")
     (instances
-      (project "H616_devboard"
+      (project "kryptokrona-mini-miner"
         (path "/44f68964-8d75-4db0-b784-705712e148bc/5d9fa4e3-c1a9-47c1-b361-a7aa11440b42"
           (reference "#PWR083") (unit 1)
@@
     (pin "1")
     (instances
-      (project "H616_devboard"
+      (project "kryptokrona-mini-miner"
         (path "/44f68964-8d75-4db0-b784-705712e148bc/5d9fa4e3-c1a9-47c1-b361-a7aa11440b42"
           (reference "#PWR067") (unit 1)
@@
     (pin "V5")
     (instances
-      (project "H616_devboard"
+      (project "kryptokrona-mini-miner"
         (path "/44f68964-8d75-4db0-b784-705712e148bc/5d9fa4e3-c1a9-47c1-b361-a7aa11440b42"
           (reference "U1") (unit 3)
@@
     (pin "2")
     (instances
-      (project "H616_devboard"
+      (project "kryptokrona-mini-miner"
         (path "/44f68964-8d75-4db0-b784-705712e148bc/5d9fa4e3-c1a9-47c1-b361-a7aa11440b42"
           (reference "C62") (unit 1)
